Commit message: kinect added

File: sim_model/urdf/sim_model.urdf.xacro (robot description, xacro)
@@ -32,4 +32,28 @@
     </inertial>
   </link>
+<!-- Defining the robot base back -->
+  <link name="base_back">
+    <visual>
+      <origin rpy="0 0 0" xyz="0 0 ${base_z}"/>
+      <geometry>
+        <box size="0.20 0.6 0.8"/>
+      </geometry>
+      <material name="white"/>
+    </visual>
+    <collision>
+      <geometry>
+        <box size="1 0.2 1"/>
+      </geometry>
+    </collision>
+    <inertial>
+      <mass value="10"/>
+      <inertia ixx="1.0" ixy="0.0" ixz="0.0" iyy="1.0" iyz="0.0" izz="1.0"/>
+    </inertial>
+  </link>
+  <joint name="base_back_joint" type="fixed">
+    <parent link="base_link"/>
+    <child link="base_back"/>
+    <origin xyz="-0.40 0 0.50"/>
+  </joint>
 <!-- Defining the robot rear wheels -->
   <xacro:macro name="rear_wheel" params="prefix suffix reflect">
@@ -61,4 +85,24 @@
       <!-- <origin xyz="${baselen*reflect/3} 0 -${wheeldiam/2+.05}" rpy="0 0 0"/> -->
     </joint>
+    <!-- This block provides the simulator (Gazebo) with information on a few additional
+    physical properties. See http://gazebosim.org/tutorials/?tut=ros_urdf for more-->
+    <gazebo reference="${prefix}_${suffix}_wheel">
+      <mu1 value="200.0"/>
+      <mu2 value="100.0"/>
+      <kp value="10000000.0" />
+      <kd value="1.0" />
+      <material>Gazebo/Grey</material>
+    </gazebo>
+    <!-- This block connects the wheel joint to an actuator (motor), which informs both
+    simulation and visualization of the robot -->
+    <transmission name="${prefix}_${suffix}_wheel_trans">
+      <type>transmission_interface/SimpleTransmission</type>
+      <actuator name="${prefix}_${suffix}_wheel_motor">
+        <mechanicalReduction>1</mechanicalReduction>
+      </actuator>
+      <joint name="${prefix}_${suffix}_wheel_joint">
+        <hardwareInterface>VelocityJointInterface</hardwareInterface>
+      </joint>
+    </transmission>
   </xacro:macro>
 <!-- Defining the robot front wheels -->
@@ -91,4 +135,24 @@
       <!-- <origin xyz="${baselen*reflect/3} 0 -${wheeldiam/2+.05}" rpy="0 0 0"/> -->
     </joint>
+    <!-- This block provides the simulator (Gazebo) with information on a few additional
+    physical properties. See http://gazebosim.org/tutorials/?tut=ros_urdf for more-->
+    <gazebo reference="${prefix}_${suffix}_wheel">
+      <mu1 value="200.0"/>
+      <mu2 value="100.0"/>
+      <kp value="10000000.0" />
+      <kd value="1.0" />
+      <material>Gazebo/Grey</material>
+    </gazebo>
+    <!-- This block connects the wheel joint to an actuator (motor), which informs both
+    simulation and visualization of the robot -->
+    <transmission name="${prefix}_${suffix}_wheel_trans">
+      <type>transmission_interface/SimpleTransmission</type>
+      <actuator name="${prefix}_${suffix}_wheel_motor">
+        <mechanicalReduction>1</mechanicalReduction>
+      </actuator>
+      <joint name="${prefix}_${suffix}_wheel_joint">
+        <hardwareInterface>VelocityJointInterface</hardwareInterface>
+      </joint>
+    </transmission>
   </xacro:macro>
   <!-- Setting the rear right wheel -->
@@ -100,4 +164,124 @@
   <!-- Setting the front left wheel -->
   <xacro:front_wheel prefix="left" suffix="front" reflect="1" />
+  <!-- Kinect definition -->
+  <gazebo reference="camera_depth_frame">
+    <sensor name="camera1" type="depth">
+      <always_on>true</always_on>
+      <update_rate>20.0</update_rate>
+      <camera>
+        <horizontal_fov>1.0471975512</horizontal_fov>
+        <image>
+          <format>R8G8B8</format>
+          <width>640</width>
+          <height>480</height>
+        </image>
+        <clip>
+          <near>0.05</near>
+          <far>8.0</far>
+        </clip>
+      </camera>
+      <plugin filename="libgazebo_ros_openni_kinect.so" name="camera_depth_frame_kinect_controller">
+        <baseline>0.1</baseline>
+        <alwaysOn>true</alwaysOn>
+        <updateRate>10</updateRate>
+        <cameraName>camera1</cameraName>
+        <imageTopicName>depth/image_raw</imageTopicName>
+        <cameraInfoTopicName>depth/camera_info</cameraInfoTopicName>
+        <depthImageTopicName>depth/image_raw</depthImageTopicName>
+        <depthImageCameraInfoTopicName>depth/camera_info</depthImageCameraInfoTopicName>
+        <pointCloudTopicName>depth/points</pointCloudTopicName>
+        <frameName>camera_depth_optical_frame</frameName>
+        <pointCloudCutoff>0.3</pointCloudCutoff>
+        <distortion_k1>0.0</distortion_k1>
+        <distortion_k2>0.0</distortion_k2>
+        <distortion_k3>0.0</distortion_k3>
+        <distortion_t1>0.0</distortion_t1>
+        <distortion_t2>0.0</distortion_t2>
+        <!--
+        <CxPrime>0</CxPrime>
+        <Cx>0</Cx>
+        <Cy>0</Cy>
+        <focalLength>0</focalLength>
+        <hackBaseline>0</hackBaseline>
+        -->
+      </plugin>
+    </sensor>
+  </gazebo>
+  <!-- Parameterised in part by the values in kinect_properties.urdf.xacro -->
+  <joint name="camera_rgb_joint" type="fixed">
+    <origin rpy="0 0 0" xyz="-0.30 0.2 0.95"/>
+    <parent link="base_link"/>
+    <child link="camera_rgb_frame"/>
+  </joint>
+  <link name="camera_rgb_frame">
+    <inertial>
+      <mass value="0.001"/>
+      <origin xyz="0 0 0"/>
+      <inertia ixx="0.0001" ixy="0.0" ixz="0.0" iyy="0.0001" iyz="0.0" izz="0.0001"/>
+    </inertial>
+  </link>
+  <joint name="camera_rgb_optical_joint" type="fixed">
+    <origin rpy="-1.57079632679 0 -1.57079632679" xyz="0 0 0"/>
+    <parent link="camera_rgb_frame"/>
+    <child link="camera_rgb_optical_frame"/>
+  </joint>
+  <link name="camera_rgb_optical_frame">
+    <inertial>
+      <mass value="0.001"/>
+      <origin xyz="0 0 0"/>
+      <inertia ixx="0.0001" ixy="0.0" ixz="0.0" iyy="0.0001" iyz="0.0" izz="0.0001"/>
+    </inertial>
+  </link>
+  <joint name="camera_joint" type="fixed">
+    <origin rpy="0 0 0" xyz="-0.031 -0.0 -0.016"/>
+    <parent link="camera_rgb_frame"/>
+    <child link="camera_link"/>
+  </joint>
+  <link name="camera_link">
+    <visual>
+      <origin rpy="0 0 1.57079632679" xyz="0 0 0"/>
+      <geometry>
+        <mesh filename="package://robot_cognition_system/sim_model/meshes/kinect.dae"/>
+      </geometry>
+    </visual>
+    <collision>
+      <origin rpy="0 0 0" xyz="0.0 0.0 0.0"/>
+      <geometry>
+        <box size="0.07271 0.27794 0.073"/>
+      </geometry>
+    </collision>
+    <inertial>
+      <mass value="0.001"/>
+      <origin xyz="0 0 0"/>
+      <inertia ixx="0.0001" ixy="0.0" ixz="0.0" iyy="0.0001" iyz="0.0" izz="0.0001"/>
+    </inertial>
+  </link>
+  <!-- The fixed joints & links below are usually published by static_transformers launched by the OpenNi launch
+		 files. However, for Gazebo simulation we need them, so we add them here.
+		 (Hence, don't publish them additionally!) -->
+  <joint name="camera_depth_joint" type="fixed">
+    <origin rpy="0 0 0" xyz="0 0.0 0"/>
+    <parent link="camera_rgb_frame"/>
+    <child link="camera_depth_frame"/>
+  </joint>
+  <link name="camera_depth_frame">
+    <inertial>
+      <mass value="0.001"/>
+      <origin xyz="0 0 0"/>
+      <inertia ixx="0.0001" ixy="0.0" ixz="0.0" iyy="0.0001" iyz="0.0" izz="0.0001"/>
+    </inertial>
+  </link>
+  <joint name="camera_depth_optical_joint" type="fixed">
+    <origin rpy="-1.57079632679 0 -1.57079632679" xyz="0 0 0"/>
+    <parent link="camera_depth_frame"/>
+    <child link="camera_depth_optical_frame"/>
+  </joint>
+  <link name="camera_depth_optical_frame">
+    <inertial>
+      <mass value="0.001"/>
+      <origin xyz="0 0 0"/>
+      <inertia ixx="0.0001" ixy="0.0" ixz="0.0" iyy="0.0001" iyz="0.0" izz="0.0001"/>
+    </inertial>
+  </link>
 <!-- Gazebo plugin for ROS Control -->
   <gazebo>

Commit message: model kinect update

File: sim_model/urdf/sim_model.urdf.xacro (robot description, xacro)
@@ -186,11 +186,12 @@
         <updateRate>10</updateRate>
         <cameraName>camera1</cameraName>
-        <imageTopicName>depth/image_raw</imageTopicName>
-        <cameraInfoTopicName>depth/camera_info</cameraInfoTopicName>
-        <depthImageTopicName>depth/image_raw</depthImageTopicName>
-        <depthImageCameraInfoTopicName>depth/camera_info</depthImageCameraInfoTopicName>
-        <pointCloudTopicName>depth/points</pointCloudTopicName>
+        <imageTopicName>/camera/color/image_raw</imageTopicName>
+        <cameraInfoTopicName>/camera/color/camera_info</cameraInfoTopicName>
+        <depthImageTopicName>/camera/depth/image_raw</depthImageTopicName>
+        <depthImageCameraInfoTopicName>/camera/depth/camera_info</depthImageCameraInfoTopicName>
+        <pointCloudTopicName>/camera/depth/points</pointCloudTopicName>
         <frameName>camera_depth_optical_frame</frameName>
-        <pointCloudCutoff>0.3</pointCloudCutoff>
+        <pointCloudCutoff>0.5</pointCloudCutoff>
+        <pointCloudCutoffMax>3.0</pointCloudCutoffMax>
         <distortion_k1>0.0</distortion_k1>
         <distortion_k2>0.0</distortion_k2>
@@ -198,11 +199,9 @@
         <distortion_t1>0.0</distortion_t1>
         <distortion_t2>0.0</distortion_t2>
-        <!--
-        <CxPrime>0</CxPrime>
+        <!-- <CxPrime>0</CxPrime>
         <Cx>0</Cx>
         <Cy>0</Cy>
         <focalLength>0</focalLength>
-        <hackBaseline>0</hackBaseline>
-        -->
+        <hackBaseline>0</hackBaseline> -->
       </plugin>
     </sensor>
@@ -210,5 +209,6 @@
   <!-- Parameterised in part by the values in kinect_properties.urdf.xacro -->
   <joint name="camera_rgb_joint" type="fixed">
-    <origin rpy="0 0 0" xyz="-0.30 0.2 0.95"/>
+    <!-- <origin rpy="0 0 0" xyz="-0.30 0.2 0.95"/> -->
+    <origin rpy="0 0 0" xyz="0.50 0.2 0.15"/>
     <parent link="base_link"/>
     <child link="camera_rgb_frame"/>
@@ -240,5 +240,5 @@
   <link name="camera_link">
     <visual>
-      <origin rpy="0 0 1.57079632679" xyz="0 0 0"/>
+      <origin rpy="0.0 0 1.57079632679" xyz="0 0 0"/>
       <geometry>
         <mesh filename="package://robot_cognition_system/sim_model/meshes/kinect.dae"/>

Commit message: publish sensor pointer data as point cloud data

File: sim_model/urdf/sim_model.urdf.xacro (robot description, xacro)
@@ -284,4 +284,68 @@
     </inertial>
   </link>
+<!-- Laser Pointer Definition -->
+ <gazebo reference="hokuyo_link">
+    <sensor type="ray" name="head_hokuyo_sensor">
+      <pose>0 0 0 0 0 0</pose>
+      <visualize>false</visualize>
+      <update_rate>40</update_rate>
+      <ray>
+        <scan>
+          <horizontal>
+            <samples>720</samples>
+            <resolution>1</resolution>
+            <!-- <min_angle>-1.570796</min_angle>
+            <max_angle>1.570796</max_angle> -->
+            <min_angle>-0.01</min_angle>
+            <max_angle>0.01</max_angle>
+          </horizontal>
+        </scan>
+        <range>
+          <min>0.10</min>
+          <max>30.0</max>
+          <resolution>0.01</resolution>
+        </range>
+        <noise>
+          <type>gaussian</type>
+          <!-- Noise parameters based on published spec for Hokuyo laser
+               achieving "+-30mm" accuracy at range < 10m.  A mean of 0.0m and
+               stddev of 0.01m will put 99.7% of samples within 0.03m of the true
+               reading. -->
+          <mean>0.0</mean>
+          <stddev>0.01</stddev>
+        </noise>
+      </ray>
+      <plugin name="gazebo_ros_head_hokuyo_controller" filename="libgazebo_ros_laser.so">
+        <topicName>/laser/pointer</topicName>
+        <frameName>hokuyo_link</frameName>
+      </plugin>
+    </sensor>
+  </gazebo>
+  <joint name="hokuyo_joint" type="fixed">
+    <axis xyz="0 1 0" />
+    <!-- <origin xyz="0 0 ${height3 - axel_offset/2}" rpy="0 0 0"/> -->
+    <origin xyz="0.50 0.0 0.15" rpy="0 0 0"/>
+    <parent link="base_link"/>
+    <child link="hokuyo_link"/>
+  </joint>
+  <link name="hokuyo_link">
+    <collision>
+      <origin xyz="0 0 0" rpy="0 0 0"/>
+      <geometry>
+    <box size="0.1 0.1 0.1"/>
+      </geometry>
+    </collision>
+    <visual>
+      <origin xyz="0 0 0" rpy="0 0 0"/>
+      <geometry>
+        <mesh filename="package://robot_cognition_system/sim_model/meshes/hokuyo.dae"/>
+      </geometry>
+    </visual>
+    <inertial>
+      <mass value="1e-5" />
+      <origin xyz="0 0 0" rpy="0 0 0"/>
+      <inertia ixx="1e-6" ixy="0" ixz="0" iyy="1e-6" iyz="0" izz="1e-6" />
+    </inertial>
+  </link>
 <!-- Gazebo plugin for ROS Control -->
   <gazebo>

Commit message: staring laser pan & tilt

File: sim_model/urdf/sim_model.urdf.xacro (robot description, xacro)
@@ -322,7 +322,8 @@
     </sensor>
   </gazebo>
-  <joint name="hokuyo_joint" type="fixed">
-    <axis xyz="0 1 0" />
+  <joint name="hokuyo_joint" type="revolute">
+    <axis xyz="0 1 1" />
     <!-- <origin xyz="0 0 ${height3 - axel_offset/2}" rpy="0 0 0"/> -->
+    <limit lower="-${3.15/2}" upper="${3.15/2}"  effort="50" velocity="1"/>
     <origin xyz="0.50 0.0 0.15" rpy="0 0 0"/>
     <parent link="base_link"/>
@@ -337,5 +338,5 @@
     </collision>
     <visual>
-      <origin xyz="0 0 0" rpy="0 0 0"/>
+      <origin xyz="0 0 0" rpy="0 0.0 0.0"/>
       <geometry>
         <mesh filename="package://robot_cognition_system/sim_model/meshes/hokuyo.dae"/>
@@ -348,4 +349,13 @@
     </inertial>
   </link>
+<!-- Laser Pan & Tilt actuator -->
+<transmission name="pan_trans">
+  <type>transmission_interface/SimpleTransmission</type>
+  <joint name="hokuyo_joint"/>
+  <actuator name="laser_pan_unit">
+    <hardwareInterface>EffortJointInterface</hardwareInterface>
+    <mechanicalReduction>1</mechanicalReduction>
+  </actuator>
+</transmission>
 <!-- Gazebo plugin for ROS Control -->
   <gazebo>

Commit message: pan join state update

File: sim_model/urdf/sim_model.urdf.xacro (robot description, xacro)
@@ -323,10 +323,18 @@
   </gazebo>
   <joint name="hokuyo_joint" type="revolute">
-    <axis xyz="0 1 1" />
+    <axis xyz="0 1 0" />
+    <!-- <origin xyz="0 0 ${height3 - axel_offset/2}" rpy="0 0 0"/> -->
+    <limit lower="-${3.15/2}" upper="${3.15/2}"  effort="50" velocity="1"/>
+    <origin xyz="0.0 0.0 0.0" rpy="0 0 0"/>
+    <parent link="hokuyo_base_link"/>
+    <child link="hokuyo_link"/>
+  </joint>
+  <joint name="hokuyo_joint_pan" type="revolute">
+    <axis xyz="0 0 1" />
     <!-- <origin xyz="0 0 ${height3 - axel_offset/2}" rpy="0 0 0"/> -->
     <limit lower="-${3.15/2}" upper="${3.15/2}"  effort="50" velocity="1"/>
     <origin xyz="0.50 0.0 0.15" rpy="0 0 0"/>
     <parent link="base_link"/>
-    <child link="hokuyo_link"/>
+    <child link="hokuyo_base_link"/>
   </joint>
   <link name="hokuyo_link">
@@ -349,13 +357,41 @@
     </inertial>
   </link>
+  <link name="hokuyo_base_link">
+    <visual>
+      <origin rpy="0 0 0" xyz="0 0 0"/>
+      <geometry>
+        <box size="0.02 0.02 0.02"/>
+      </geometry>
+      <material name="black"/>
+    </visual>
+    <collision>
+      <geometry>
+        <box size="0.02 0.02 0.02"/>
+      </geometry>
+    </collision>
+    <inertial>
+      <mass value="1"/>
+      <inertia ixx="1.0" ixy="0.0" ixz="0.0" iyy="1.0" iyz="0.0" izz="1.0"/>
+    </inertial>
+  </link>
+  <transmission name="laser_trans">
+    <type>transmission_interface/SimpleTransmission</type>
+    <actuator name="laser_motor">
+      <mechanicalReduction>1</mechanicalReduction>
+    </actuator>
+    <joint name="hokuyo_joint">
+      <hardwareInterface>PositionJointInterface</hardwareInterface>
+    </joint>
+  </transmission>
 <!-- Laser Pan & Tilt actuator -->
-<transmission name="pan_trans">
-  <type>transmission_interface/SimpleTransmission</type>
-  <joint name="hokuyo_joint"/>
-  <actuator name="laser_pan_unit">
-    <hardwareInterface>EffortJointInterface</hardwareInterface>
-    <mechanicalReduction>1</mechanicalReduction>
-  </actuator>
-</transmission>
+  <transmission name="laser_trans_pan">
+    <type>transmission_interface/SimpleTransmission</type>
+    <actuator name="laser_motor_pan">
+      <mechanicalReduction>1</mechanicalReduction>
+    </actuator>
+    <joint name="hokuyo_joint_pan">
+      <hardwareInterface>PositionJointInterface</hardwareInterface>
+    </joint>
+  </transmission>
 <!-- Gazebo plugin for ROS Control -->
   <gazebo>

Commit message: pan tilt control via Web

File: sim_model/urdf/sim_model.urdf.xacro (robot description, xacro)
@@ -288,5 +288,5 @@
     <sensor type="ray" name="head_hokuyo_sensor">
       <pose>0 0 0 0 0 0</pose>
-      <visualize>false</visualize>
+      <visualize>true</visualize>
       <update_rate>40</update_rate>
       <ray>
@@ -371,11 +371,11 @@
     </collision>
     <inertial>
-      <mass value="1"/>
-      <inertia ixx="1.0" ixy="0.0" ixz="0.0" iyy="1.0" iyz="0.0" izz="1.0"/>
-    </inertial>
-  </link>
-  <transmission name="laser_trans">
+      <mass value="0.001"/>
+      <inertia ixx="0.0001" ixy="0.0" ixz="0.0" iyy="0.0001" iyz="0.0" izz="0.0001"/>
+    </inertial>
+  </link>
+  <transmission name="laser_trans_tilt">
     <type>transmission_interface/SimpleTransmission</type>
-    <actuator name="laser_motor">
+    <actuator name="laser_motor_tilt">
       <mechanicalReduction>1</mechanicalReduction>
     </actuator>
@@ -384,5 +384,4 @@
     </joint>
   </transmission>
-<!-- Laser Pan & Tilt actuator -->
   <transmission name="laser_trans_pan">
     <type>transmission_interface/SimpleTransmission</type>

Commit message: classifier review sync

File: sim_model/urdf/sim_model.urdf.xacro (robot description, xacro)
@@ -322,5 +322,5 @@
     </sensor>
   </gazebo>
-  <joint name="hokuyo_joint" type="revolute">
+  <joint name="hokuyo_joint" type="continuous">
     <axis xyz="0 1 0" />
     <!-- <origin xyz="0 0 ${height3 - axel_offset/2}" rpy="0 0 0"/> -->
@@ -330,5 +330,5 @@
     <child link="hokuyo_link"/>
   </joint>
-  <joint name="hokuyo_joint_pan" type="revolute">
+  <joint name="hokuyo_joint_pan" type="continuous">
     <axis xyz="0 0 1" />
     <!-- <origin xyz="0 0 ${height3 - axel_offset/2}" rpy="0 0 0"/> -->
@@ -371,6 +371,7 @@
     </collision>
     <inertial>
-      <mass value="0.001"/>
-      <inertia ixx="0.0001" ixy="0.0" ixz="0.0" iyy="0.0001" iyz="0.0" izz="0.0001"/>
+      <mass value="1e-5" />
+      <origin xyz="0 0 0" rpy="0 0 0"/>
+      <inertia ixx="1e-6" ixy="0" ixz="0" iyy="1e-6" iyz="0" izz="1e-6" />
     </inertial>
   </link>

Commit message: laser postion adjustment

File: sim_model/urdf/sim_model.urdf.xacro (robot description, xacro)
@@ -325,5 +325,5 @@
     <axis xyz="0 1 0" />
     <!-- <origin xyz="0 0 ${height3 - axel_offset/2}" rpy="0 0 0"/> -->
-    <limit lower="-${3.15/2}" upper="${3.15/2}"  effort="50" velocity="1"/>
+    <limit lower="-${3.1}" upper="${3.1}"  effort="50" velocity="1"/>
     <origin xyz="0.0 0.0 0.0" rpy="0 0 0"/>
     <parent link="hokuyo_base_link"/>
@@ -334,5 +334,5 @@
     <!-- <origin xyz="0 0 ${height3 - axel_offset/2}" rpy="0 0 0"/> -->
     <limit lower="-${3.15/2}" upper="${3.15/2}"  effort="50" velocity="1"/>
-    <origin xyz="0.50 0.0 0.15" rpy="0 0 0"/>
+    <origin xyz="0.50 -0.20 0.15" rpy="0 0 0"/>
     <parent link="base_link"/>
     <child link="hokuyo_base_link"/>
