Commit message: castor wheel implementation

File: sim_model/urdf/sim_model.urdf.xacro (robot description, xacro)
@@ -1,4 +1,37 @@
 <?xml version="1.0"?>
+<!-- The castor wheel functionality - Credits for the Toronto Robotics Clud
+  https://github.com/Toronto-Robotics-club/Gazebo_caster_sample/blob/master/jimmy_description/urdf/jimmy.xacro
+ -->
 <robot name="macroed" xmlns:xacro="http://ros.org/wiki/xacro">
+  <xacro:property name="pi" value="3.1415926535897931" />
+  <!--base link values-->
+  <xacro:property name="base_link_length_width_height" value="0.650 0.381 0.132" />
+  <xacro:property name="base_link_length" value="1" />
+  <xacro:property name="base_link_width" value="0.7" />
+  <xacro:property name="base_link_height" value="0.2" />
+  <xacro:property name="base_link_mass" value="20"/> <!--25 kg-->
+  <!--left and right castor mount plate size (both are same size)-->
+  <xacro:property name="castor_mount_link_length_width_height" value="0.1145 0.10 0.0057" />
+  <xacro:property name="castor_mount_link_length" value="0.1145" />
+  <xacro:property name="castor_mount_link_width" value="0.10" />
+  <xacro:property name="castor_mount_link_height" value="0.0057" />
+  <xacro:property name="castor_mount_link_mass" value="0.25"/> <!--0.25 kg-->
+  <!--dummy link to give castors rotation about the Z axis-->
+  <xacro:property name="castor_mount_dummy_link_length" value="0.02" />
+  <xacro:property name="castor_mount_dummy_link_width" value="0.02" />
+  <xacro:property name="castor_mount_dummy_link_height" value="0.02" />
+  <xacro:property name="castor_mount_dummy_link_mass" value="1.5"/> <!--0.25 kg-->
+  <!--Friction for joints-->
+  <xacro:property name="friction_val" value="0.15"/>
+  <!--Other properties-->
+  <xacro:property name="rear_wheel_radius" value="0.15" />
+  <xacro:property name="front_wheel_radius" value="0.10" />
+  <xacro:property name="rear_wheel_length" value="0.1" />
+  <xacro:property name="front_wheel_length" value="0.1" />
+  <xacro:property name="rear_wheel_mass" value="8" />
+  <xacro:property name="front_wheel_mass" value="5" />
+  <xacro:property name="base_z" value="0" />
+  <xacro:property name="joint_friction" value="0.15" />
+  <xacro:property name="joint_castor_friction" value="0.15" />
 <!-- Material colors definition -->
   <material name="white">
@@ -8,9 +41,4 @@
     <color rgba="0 0 0 1"/>
   </material>
-<!-- Properties definitions -->
-  <xacro:property name="rear_wheel_radius" value="0.15" />
-  <xacro:property name="front_wheel_radius" value="0.10" />
-  <xacro:property name="base_z" value="0" />
-  <!-- <xacro:property name="base_z" value="0.32" /> -->
 <!-- Defining the robot base -->
   <link name="base_link">
@@ -28,6 +56,14 @@
     </collision>
     <inertial>
-      <mass value="10"/>
-      <inertia ixx="1.0" ixy="0.0" ixz="0.0" iyy="1.0" iyz="0.0" izz="1.0"/>
+      <mass value="${base_link_mass}"/>
+      <!--This is the 3x3 inertial matrix. See: https://wiki.ros.org/urdf/XML/link -->
+      <!--where x=length; y=width; z=height. these lines of code came from Emiliano Borghi's project-->
+      <inertia
+        ixx="${base_link_mass*(base_link_width*base_link_width+base_link_height*base_link_height)/12}"
+        ixy="0"
+        ixz="0"
+        iyy="${base_link_mass*(base_link_length*base_link_length+base_link_height*base_link_height)/12}"
+        iyz="0"
+        izz="${base_link_mass*(base_link_length*base_link_length+base_link_height*base_link_height)/12}"/>
     </inertial>
   </link>
@@ -57,10 +93,10 @@
   </joint>
 <!-- Defining the robot rear wheels -->
-  <xacro:macro name="rear_wheel" params="prefix suffix reflect">
+  <xacro:macro name="rear_wheel" params="prefix suffix reflect mass radius length">
     <link name="${prefix}_${suffix}_wheel">
       <visual>
         <origin xyz="0 0 ${base_z}" rpy="${pi/2} 0 0" />
         <geometry>
-          <cylinder radius="${rear_wheel_radius}" length="0.1"/>
+          <cylinder radius="${radius}" length="${length}"/>
         </geometry>
         <material name="black"/>
@@ -68,12 +104,24 @@
       <collision>
         <geometry>
-          <cylinder radius="${rear_wheel_radius}" length="0.1"/>
+          <cylinder radius="${radius}" length="${length}"/>
         </geometry>
         <origin xyz="0 0 ${base_z}" rpy="${pi/2} 0 0" />
       </collision>
       <inertial>
+        <mass value="${mass}"/>
+        <!--This is the 3x3 inertial matrix. See: https://wiki.ros.org/urdf/XML/link -->
+        <inertia
+            ixx="${mass*(3*radius*radius+length*length)/12}"
+            ixy = "0"
+            ixz = "0"
+            iyy="${mass*(3*radius*radius+length*length)/12}"
+            iyz = "0"
+            izz="${mass*radius*radius/2}"
+          />
+      </inertial>
+      <!-- <inertial>
         <mass value="10"/>
         <inertia ixx="1.0" ixy="0.0" ixz="0.0" iyy="1.0" iyz="0.0" izz="1.0"/>
-      </inertial>
+      </inertial> -->
       <!-- <xacro:default_inertial mass="1"/> -->
     </link>
@@ -83,4 +131,5 @@
       <child link="${prefix}_${suffix}_wheel"/>
       <origin xyz="${-0.35} ${reflect*0.4} ${-0.17}"/>
+      <dynamics damping="0.0" friction="${joint_friction}"/>
       <!-- <origin xyz="${baselen*reflect/3} 0 -${wheeldiam/2+.05}" rpy="0 0 0"/> -->
     </joint>
@@ -107,10 +156,10 @@
   </xacro:macro>
 <!-- Defining the robot front wheels -->
-  <xacro:macro name="front_wheel" params="prefix suffix reflect">
+  <xacro:macro name="front_wheel" params="prefix suffix reflect mass radius length">
     <link name="${prefix}_${suffix}_wheel">
       <visual>
         <origin xyz="0 0 ${base_z}" rpy="${pi/2} 0 0" />
         <geometry>
-          <cylinder radius="${front_wheel_radius}" length="0.1"/>
+          <cylinder radius="${radius}" length="${radius}"/>
         </geometry>
         <material name="black"/>
@@ -118,19 +167,27 @@
       <collision>
         <geometry>
-          <cylinder radius="${front_wheel_radius}" length="0.1"/>
+          <cylinder radius="${radius}" length="${radius}"/>
         </geometry>
         <origin xyz="0 0 ${base_z}" rpy="${pi/2} 0 0" />
       </collision>
       <inertial>
-        <mass value="10"/>
-        <inertia ixx="1.0" ixy="0.0" ixz="0.0" iyy="1.0" iyz="0.0" izz="1.0"/>
+        <mass value="${mass}"/>
+        <!--This is the 3x3 inertial matrix. See: https://wiki.ros.org/urdf/XML/link -->
+        <inertia
+            ixx="${mass*(3*radius*radius+length*length)/12}"
+            ixy = "0"
+            ixz = "0"
+            iyy="${mass*(3*radius*radius+length*length)/12}"
+            iyz = "0"
+            izz="${mass*radius*radius/2}"
+          />
       </inertial>
-      <!-- <xacro:default_inertial mass="1"/> -->
     </link>
     <joint name="${prefix}_${suffix}_wheel_joint" type="continuous">
       <axis xyz="0 1 0" rpy="0 0 0" />
-      <parent link="base_link"/>
+      <parent link="${prefix}_castor_dummy"/>
       <child link="${prefix}_${suffix}_wheel"/>
-      <origin xyz="${0.35} ${reflect*0.35} ${-0.22}"/>
+      <origin xyz="0 0 -0.12"/>
+      <dynamics damping="0.0" friction="${joint_friction}"/>
       <!-- <origin xyz="${baselen*reflect/3} 0 -${wheeldiam/2+.05}" rpy="0 0 0"/> -->
     </joint>
@@ -156,12 +213,115 @@
     </transmission>
   </xacro:macro>
+  <!-- Defining the castor mount -->
+  <xacro:macro name="castor_mount" params="prefix reflect length width height material mass">
+    <link name="${prefix}_castor_mount">
+      <collision>
+        <geometry>
+          <box size="${length} ${width} ${height}"/>
+        </geometry>
+        <origin xyz="0 0 ${base_z}" rpy="${pi/2} 0 0" />
+      </collision>
+      <visual>
+        <geometry>
+          <box size="${length} ${width} ${height}"/>
+        </geometry>
+        <origin xyz="0 0 ${base_z}" rpy="0 0 0" />
+        <material name="${material}"/>
+      </visual>
+      <inertial>
+        <origin xyz="0 0 ${base_z}" rpy="0 0 0" />
+        <mass value="${mass}"/>
+        <!--This is the 3x3 inertial matrix. See: https://wiki.ros.org/urdf/XML/link -->
+        <!--where x=length; y=width; z=height. these lines of code came from
+        Emiliano Borghi's project-->
+        <inertia
+          ixx="${mass*(width*width+height*height)/12}"
+    	    ixy = "0"
+    	    ixz = "0"
+    	    iyy="${mass*(length*length+height*height)/12}"
+    	    iyz = "0"
+    	    izz="${mass*(length*length+height*height)/12}"/>
+      </inertial>
+    </link>
+    <joint name="${prefix}_castor_mount_joint" type="fixed">
+      <axis xyz="0 1 0" rpy="0 0 0" />
+      <parent link="base_link"/>
+      <child link="${prefix}_castor_mount"/>
+      <origin xyz="${0.35} ${reflect*0.30} ${-0.10}"/>
+      <!-- <origin xyz="${baselen*reflect/3} 0 -${wheeldiam/2+.05}" rpy="0 0 0"/> -->
+    </joint>
+  </xacro:macro>
+  <!-- Defining the castor dummy for Z axis rotation -->
+  <xacro:macro name="castor_dummy" params="prefix reflect length width height material mass">
+    <link name="${prefix}_castor_dummy">
+      <collision>
+        <geometry>
+          <box size="${length} ${width} ${height}"/>
+        </geometry>
+        <origin xyz="0 0 ${base_z}" rpy="${pi/2} 0 0" />
+      </collision>
+      <visual>
+        <geometry>
+          <box size="${length} ${width} ${height}"/>
+        </geometry>
+        <origin xyz="0 0 ${base_z}" rpy="0 0 0" />
+        <material name="${material}"/>
+      </visual>
+      <inertial>
+        <origin xyz="0 0 ${base_z}" rpy="0 0 0" />
+        <mass value="${mass}"/>
+        <!--This is the 3x3 inertial matrix. See: https://wiki.ros.org/urdf/XML/link -->
+        <!--where x=length; y=width; z=height. these lines of code came from
+        Emiliano Borghi's project-->
+        <inertia
+          ixx="${mass*(width*width+height*height)/12}"
+    	    ixy = "0"
+    	    ixz = "0"
+    	    iyy="${mass*(length*length+height*height)/12}"
+    	    iyz = "0"
+    	    izz="${mass*(length*length+height*height)/12}"/>
+      </inertial>
+    </link>
+    <joint name="${prefix}_castor_dummy_joint" type="continuous">
+      <axis xyz="0 0 1" rpy="0 0 0" />
+      <parent link="${prefix}_castor_mount"/>
+      <child link="${prefix}_castor_dummy"/>
+      <origin xyz="0 0 -0.01"/>
+      <dynamics damping="0.0" friction="${joint_castor_friction}"/>
+      <!-- <origin xyz="${baselen*reflect/3} 0 -${wheeldiam/2+.05}" rpy="0 0 0"/> -->
+    </joint>
+  </xacro:macro>
   <!-- Setting the rear right wheel -->
-  <xacro:rear_wheel prefix="right" suffix="rear" reflect="-1" />
+  <xacro:rear_wheel prefix="right" suffix="rear" reflect="-1" mass="${rear_wheel_mass}" radius="${rear_wheel_radius}" length="${rear_wheel_length}"/>
   <!-- Setting the rear left wheel -->
-  <xacro:rear_wheel prefix="left" suffix="rear" reflect="1" />
+  <xacro:rear_wheel prefix="left" suffix="rear" reflect="1" mass="${rear_wheel_mass}"  radius="${rear_wheel_radius}" length="${rear_wheel_length}"/>
+  <!-- Setting the castor mount left wheel -->
+  <xacro:castor_mount prefix="left" reflect="1" length="${castor_mount_link_length}"
+                                                width="${castor_mount_link_width}"
+                                                height="${castor_mount_link_height}"
+                                                material="white"
+                                                mass="${castor_mount_link_mass}"/>
+  <!-- Setting the castor mount right wheel -->
+  <xacro:castor_mount prefix="right" reflect="-1" length="${castor_mount_link_length}"
+                                                width="${castor_mount_link_width}"
+                                                height="${castor_mount_link_height}"
+                                                material="white"
+                                                mass="${castor_mount_link_mass}"/>
+  <!-- Setting the castor dummy left wheel -->
+  <xacro:castor_dummy prefix="left" reflect="1" length="${castor_mount_dummy_link_length}"
+                                                width="${castor_mount_dummy_link_width}"
+                                                height="${castor_mount_dummy_link_height}"
+                                                material="orange"
+                                                mass="${castor_mount_dummy_link_mass}"/>
+  <!-- Setting the castor dummy left wheel -->
+  <xacro:castor_dummy prefix="right" reflect="-1" length="${castor_mount_dummy_link_length}"
+                                                width="${castor_mount_dummy_link_width}"
+                                                height="${castor_mount_dummy_link_height}"
+                                                material="orange"
+                                                mass="${castor_mount_dummy_link_mass}"/>
   <!-- Setting the front right wheel -->
-  <xacro:front_wheel prefix="right" suffix="front" reflect="-1" />
+  <xacro:front_wheel prefix="right" suffix="front" reflect="-1" mass="${front_wheel_mass}"  radius="${front_wheel_radius}" length="${front_wheel_length}"/>
   <!-- Setting the front left wheel -->
-  <xacro:front_wheel prefix="left" suffix="front" reflect="1" />
+  <xacro:front_wheel prefix="left" suffix="front" reflect="1" mass="${front_wheel_mass}"  radius="${front_wheel_radius}" length="${front_wheel_length}"/>
   <!-- Kinect definition -->
   <gazebo reference="camera_depth_frame">

Commit message: move to target updates

File: sim_model/urdf/sim_model.urdf.xacro (robot description, xacro)
@@ -283,10 +283,10 @@
       </inertial>
     </link>
-    <joint name="${prefix}_castor_dummy_joint" type="continuous">
+    <joint name="${prefix}_castor_dummy_joint" type="fixed">
       <axis xyz="0 0 1" rpy="0 0 0" />
       <parent link="${prefix}_castor_mount"/>
       <child link="${prefix}_castor_dummy"/>
       <origin xyz="0 0 -0.01"/>
-      <dynamics damping="0.0" friction="${joint_castor_friction}"/>
+      <!-- <dynamics damping="0.0" friction="${joint_castor_friction}"/>  -->
       <!-- <origin xyz="${baselen*reflect/3} 0 -${wheeldiam/2+.05}" rpy="0 0 0"/> -->
     </joint>
@@ -558,4 +558,6 @@
     <plugin name="gazebo_ros_control" filename="libgazebo_ros_control.so">
       <robotNamespace>/</robotNamespace>
+      <robotSimType>gazebo_ros_control/DefaultRobotHWSim</robotSimType>
+      <legacyModeNS>true</legacyModeNS>
     </plugin>
   </gazebo>

Commit message: friction review

File: sim_model/urdf/sim_model.urdf.xacro (robot description, xacro)
@@ -83,5 +83,5 @@
     </collision>
     <inertial>
-      <mass value="10"/>
+      <mass value="15"/>
       <inertia ixx="1.0" ixy="0.0" ixz="0.0" iyy="1.0" iyz="0.0" izz="1.0"/>
     </inertial>
@@ -132,4 +132,5 @@
       <origin xyz="${-0.35} ${reflect*0.4} ${-0.17}"/>
       <dynamics damping="0.0" friction="${joint_friction}"/>
+      <!-- <limit effort="5" velocity="5"/> -->
       <!-- <origin xyz="${baselen*reflect/3} 0 -${wheeldiam/2+.05}" rpy="0 0 0"/> -->
     </joint>
@@ -137,8 +138,8 @@
     physical properties. See http://gazebosim.org/tutorials/?tut=ros_urdf for more-->
     <gazebo reference="${prefix}_${suffix}_wheel">
-      <mu1 value="200.0"/>
-      <mu2 value="100.0"/>
-      <kp value="10000000.0" />
-      <kd value="1.0" />
+      <mu1 value="0.5"/>
+      <mu2 value="0.5"/>
+      <!-- <kp value="10000000.0" />
+      <kd value="1.0" /> -->
       <material>Gazebo/Grey</material>
     </gazebo>
@@ -190,4 +191,5 @@
       <origin xyz="0 0 -0.12"/>
       <dynamics damping="0.0" friction="${joint_friction}"/>
+      <!-- <limit effort="2" velocity="2"/> -->
       <!-- <origin xyz="${baselen*reflect/3} 0 -${wheeldiam/2+.05}" rpy="0 0 0"/> -->
     </joint>
@@ -195,8 +197,8 @@
     physical properties. See http://gazebosim.org/tutorials/?tut=ros_urdf for more-->
     <gazebo reference="${prefix}_${suffix}_wheel">
-      <mu1 value="200.0"/>
-      <mu2 value="100.0"/>
-      <kp value="10000000.0" />
-      <kd value="1.0" />
+      <mu1 value="0.5"/>
+      <mu2 value="0.5"/>
+      <!-- <kp value="10000000.0" />
+      <kd value="1.0" /> -->
       <material>Gazebo/Grey</material>
     </gazebo>
